File: hardware/kicad/pedalSHIELD_MEGA.kicad_sch (KiCad schematic)
At the start: 37 parts, among them J1 AudioJack, J2 AudioJack, SW1 SW_3PDT, SW2 SW_SPDT, SW3 SW_Push, SW4 SW_Push, U1 LT972

Commit message: kicad project update
Parts:
- A1: value Arduino_Mega_Shield -> ~
- D1: value LED -> ~
- J1, J2: value AudioJack -> ~
- LCD1: value LCD -> ~
- SW1: value SW_3PDT -> ~
- SW2: value SW_SPDT -> ~
- SW3, SW4: value SW_Push -> ~
- U1: value LT972 -> ~
Other:
- title: pedalSHIELD_MEGA -> pedalSHIELD_MEGA Schematic
