File: hardware/kicad/pedalSHIELD_MEGA.kicad_pcb (KiCad board)
At the start: 2 copper layers, 62 x 122 mm, 38 parts, among them J1 AudioJack, J2 AudioJack, SW1 SW_3PDT, SW2 SW_SPDT, SW3 SW_Push, SW4 SW_Push, U1 LT972

Commit message: kicad project update
Routing:
- net /bypass: track 12.5 -> 16.1 mm
- net /PWM_7: track 70.5 -> 71.3 mm
- net GND: vias 44 -> 45
Other:
- board text added: "ElectroSmash Nablum Rev 2.1"
- board text removed: "ElectroSmash Nablum Rev 2.0"
Changed lines of the file:
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@@
 	)
 	(paper "A4")
+	(title_block
+		(title "pedalSHIELD_MEGA PCB")
+		(date "2025-03-25")
+		(rev "2.1")
+	)
 	(layers
 		(0 "F.Cu" signal)
@@
 		(fp_arc
 			(start 100.1008 51.8922)
-			(mid 99.878928 52.516027)
+			(mid 99.878934 52.516032)
 			(end 99.542 53.086)
 			(stroke
@@
 		(layer "Edge.Cuts")
 	)
-	(gr_text "ElectroSmash\nNablum\nRev 2.0"
+	(gr_text "ElectroSmash\nNablum\nRev 2.1"
 		(at 21.5 38.75 0)
 		(layer "F.SilkS")
@@
 	)
 	(via
+		(at 42.5 118)
+		(size 0.6)
+		(drill 0.3)
+		(layers "F.Cu" "B.Cu")
+		(free yes)
+		(net 13)
+	)
+	(via
 		(at 79.75 142.75)
 		(size 0.6)
@@
 	)
 	(segment
-		(start 61.5 87.5)
-		(end 70 87.5)
+		(start 41.25 117.51)
+		(end 41.25 110.25)
 		(width 0.3)
 		(layer "F.Cu")
@@
 	)
 	(segment
-		(start 71.25 86.25)
-		(end 71.25 79.26)
+		(start 70 87.5)
+		(end 71.25 86.25)
 		(width 0.3)
 		(layer "F.Cu")
@@
 	)
 	(segment
-		(start 73.08 77.43)
-		(end 74.75 77.43)
+		(start 58 107)
+		(end 58 91)
 		(width 0.3)
 		(layer "F.Cu")
@@
 	)
 	(segment
-		(start 58 107)
-		(end 58 91)
+		(start 42.75 108.75)
+		(end 56.25 108.75)
 		(width 0.3)
 		(layer "F.Cu")
@@
 	)
 	(segment
-		(start 70 87.5)
-		(end 71.25 86.25)
+		(start 38.81 119.95)
+		(end 41.25 117.51)
 		(width 0.3)
 		(layer "F.Cu")
@@
 	)
 	(segment
-		(start 58 91)
-		(end 61.5 87.5)
+		(start 71.25 79.26)
+		(end 73.08 77.43)
 		(width 0.3)
 		(layer "F.Cu")
@@
 	)
 	(segment
-		(start 38.81 119.95)
-		(end 42.25 116.51)
+		(start 56.25 108.75)
+		(end 58 107)
 		(width 0.3)
 		(layer "F.Cu")
@@
 	)
 	(segment
-		(start 56 109)
-		(end 58 107)
+		(start 61.5 87.5)
+		(end 70 87.5)
 		(width 0.3)
 		(layer "F.Cu")
@@
 	)
 	(segment
-		(start 71.25 79.26)
-		(end 73.08 77.43)
+		(start 41.25 110.25)
+		(end 42.75 108.75)
 		(width 0.3)
 		(layer "F.Cu")
@@
 	)
 	(segment
-		(start 42.25 110.5)
-		(end 43.75 109)
+		(start 58 91)
+		(end 61.5 87.5)
 		(width 0.3)
 		(layer "F.Cu")
@@
 	)
 	(segment
-		(start 43.75 109)
-		(end 56 109)
+		(start 71.25 86.25)
+		(end 71.25 79.26)
 		(width 0.3)
 		(layer "F.Cu")
@@
 	)
 	(segment
-		(start 42.25 116.51)
-		(end 42.25 110.5)
+		(start 73.08 77.43)
+		(end 74.75 77.43)
 		(width 0.3)
 		(layer "F.Cu")
@@
 	)
 	(segment
-		(start 45.5 131.5)
+		(start 41.35 150.45)
 		(end 45.5 146.3)
 		(width 0.3)
@@
 	)
 	(segment
+		(start 47.5 116)
+		(end 50 113.5)
+		(width 0.3)
+		(layer "B.Cu")
+		(net 61)
+	)
+	(segment
 		(start 47.5 129.5)
-		(end 45.5 131.5)
+		(end 47.5 116)
 		(width 0.3)
 		(layer "B.Cu")
@@
 	)
 	(segment
-		(start 50 112.7)
-		(end 47.5 115.2)
+		(start 50 113.5)
+		(end 50 112.7)
 		(width 0.3)
 		(layer "B.Cu")
@@
 	)
 	(segment
-		(start 47.5 115.2)
+		(start 45.5 131.5)
 		(end 47.5 129.5)
 		(width 0.3)
@@
 	(segment
 		(start 45.5 146.3)
-		(end 41.35 150.45)
+		(end 45.5 131.5)
 		(width 0.3)
 		(layer "B.Cu")
@@
 	(segment
 		(start 45.2 112.7)
-		(end 47.5 115)
+		(end 43.3 112.7)
 		(width 0.3)
-		(layer "F.Cu")
+		(layer "B.Cu")
+		(net 64)
+	)
+	(segment
+		(start 41.25 121.25)
+		(end 43.3 123.3)
+		(width 0.3)
+		(layer "B.Cu")
+		(net 64)
+	)
+	(segment
+		(start 43.3 112.7)
+		(end 41.25 114.75)
+		(width 0.3)
+		(layer "B.Cu")
 		(net 64)
 	)
 	(segment
-		(start 47.5 121)
+		(start 43.3 123.3)
 		(end 45.2 123.3)
 		(width 0.3)
-		(layer "F.Cu")
+		(layer "B.Cu")
 		(net 64)
 	)
 	(segment
-		(start 47.5 115)
-		(end 47.5 121)
+		(start 41.25 114.75)
+		(end 41.25 121.25)
 		(width 0.3)
-		(layer "F.Cu")
+		(layer "B.Cu")
 		(net 64)
 	)

Commit message: rev 2.1
Parts:
- A1: value Arduino_Mega_Shield -> ~
- D1: value LED -> ~
- J1, J2: value AudioJack -> ~
- LCD1: value LCD -> ~
- SW1: value SW_3PDT -> ~
- SW2: value SW_SPDT -> ~
- SW3, SW4: value SW_Push -> ~
- U1: value LT972 -> ~

Commit message: rev 2.1
Parts:
- moved J1 2.00 mm to (33.0, 142.4)
- moved J2 2.00 mm to (67.0, 142.2)
Routing:
- net /input_jack: track 26.2 -> 24.2 mm
- net /output_jack: track 41.3 -> 42.2 mm
Changed lines of the file:
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@@
 		)
 		(pad "" np_thru_hole circle
-			(at -15.75 -14.5)
+			(at -15.3 -13.9)
 			(size 3 3)
-			(drill 3)
+			(drill 3.2)
 			(layers "F&B.Cu" "*.Mask")
 		)
 		(pad "" np_thru_hole circle
-			(at -15.75 15)
+			(at -15.3 14.7)
 			(size 3 3)
-			(drill 3)
+			(drill 3.2)
 			(layers "F&B.Cu" "*.Mask")
 		)
 		(pad "" np_thru_hole circle
-			(at 15.75 -14.5)
+			(at 15.3 -13.9)
 			(size 3 3)
-			(drill 3)
+			(drill 3.2)
 			(layers "F&B.Cu" "*.Mask")
 		)
 		(pad "" np_thru_hole circle
-			(at 15.75 15)
+			(at 15.3 14.7)
 			(size 3 3)
-			(drill 3)
+			(drill 3.2)
 			(layers "F&B.Cu" "*.Mask")
 		)
@@
 		)
 		(group ""
-			(members "5e34c4a5-05b2-4793-97b4-7d4c23198746" "6f474d3b-9059-429f-8feb-f840fb44683f"
-				"a3517b08-cab5-4f5b-9ede-fd64ee1d7600" "a4207179-764c-43b1-b26f-47c1c25264b7"
+			(members "2c19413f-a745-45bb-aaaa-5ce23453f2a2" "3e669e28-d50f-4ca3-a5ad-315075ab8fb6"
+				"d7ea7ff0-aeed-474f-8f28-88134c0c1589" "e74a00d9-eae3-4d13-9e33-2cb6ceff9b6f"
 			)
 		)
@@
 	(footprint "pedalSHIELD_MEGA:Jack_6.35mm_Neutrik_NMJ6HCD2_Horizontal"
 		(layer "F.Cu")
-		(at 65 142.22)
+		(at 67 142.22)
 		(descr "M Series, 6.35mm (1/4in) stereo jack, switched, with chrome ferrule and straight PCB pins, https://www.neutrik.com/en/product/nmj6hcd2")
 		(tags "neutrik jack m")
@@
 		(model "${KIPRJMOD}/packages3D/NMJ6HCD2.stp"
 			(offset
-				(xyz 0 0 0)
+				(xyz 0 0 1.5)
 			)
 			(scale
@@
 	(footprint "pedalSHIELD_MEGA:Jack_6.35mm_Neutrik_NMJ6HCD2_Horizontal"
 		(layer "F.Cu")
-		(at 35 142.45 180)
+		(at 33 142.45 180)
 		(descr "M Series, 6.35mm (1/4in) stereo jack, switched, with chrome ferrule and straight PCB pins, https://www.neutrik.com/en/product/nmj6hcd2")
 		(tags "neutrik jack m")
@@
 		(model "${KIPRJMOD}/packages3D/NMJ6HCD2.stp"
 			(offset
-				(xyz 0 0 0)
+				(xyz 0 0 1.5)
 			)
 			(scale
@@
 		(model "${KIPRJMOD}/packages3D/PT10LH01-101A2020.stp"
 			(offset
-				(xyz -2.25 0 7)
+				(xyz -2.25 0 9)
 			)
 			(scale
@@
 		(fp_arc
 			(start 100.1008 51.8922)
-			(mid 99.878928 52.516027)
+			(mid 99.878934 52.516032)
 			(end 99.542 53.086)
 			(stroke
@@
 	)
 	(segment
-		(start 41.35 150.45)
-		(end 45.5 146.3)
+		(start 50 113.5)
+		(end 47.5 116)
 		(width 0.3)
 		(layer "B.Cu")
@@
 	)
 	(segment
-		(start 47.5 116)
-		(end 50 113.5)
+		(start 45.5 131.5)
+		(end 45.5 144.3)
 		(width 0.3)
 		(layer "B.Cu")
@@
 	)
 	(segment
-		(start 47.5 129.5)
-		(end 47.5 116)
+		(start 47.5 116)
+		(end 47.5 129.5)
 		(width 0.3)
 		(layer "B.Cu")
@@
 	)
 	(segment
-		(start 50 113.5)
-		(end 50 112.7)
+		(start 47.5 129.5)
+		(end 45.5 131.5)
 		(width 0.3)
 		(layer "B.Cu")
@@
 	)
 	(segment
-		(start 45.5 131.5)
-		(end 47.5 129.5)
+		(start 45.5 144.3)
+		(end 39.35 150.45)
 		(width 0.3)
 		(layer "B.Cu")
@@
 	)
 	(segment
-		(start 45.5 146.3)
-		(end 45.5 131.5)
+		(start 50 112.7)
+		(end 50 113.5)
 		(width 0.3)
 		(layer "B.Cu")
@@
 	(segment
 		(start 63.4 131.85)
-		(end 62.85 132.4)
+		(end 61.03 134.22)
 		(width 0.3)
 		(layer "B.Cu")
@@
 	)
 	(segment
-		(start 50 125.8)
-		(end 51.7 127.5)
-		(width 0.3)
-		(layer "B.Cu")
-		(net 62)
-	)
-	(segment
-		(start 62.85 132.4)
-		(end 60.47 132.4)
+		(start 62.5 127.5)
+		(end 63.4 128.4)
 		(width 0.3)
 		(layer "B.Cu")
@@
 	)
 	(segment
-		(start 62.5 127.5)
-		(end 63.4 128.4)
+		(start 51.7 127.5)
+		(end 62.5 127.5)
 		(width 0.3)
 		(layer "B.Cu")
@@
 	)
 	(segment
-		(start 60.47 132.4)
-		(end 58.65 134.22)
+		(start 63.4 128.4)
+		(end 63.4 131.85)
 		(width 0.3)
 		(layer "B.Cu")
@@
 	)
 	(segment
-		(start 63.4 128.4)
-		(end 63.4 131.85)
+		(start 50 125.8)
+		(end 51.7 127.5)
 		(width 0.3)
 		(layer "B.Cu")
@@
 	)
 	(segment
-		(start 51.7 127.5)
-		(end 62.5 127.5)
+		(start 61.03 134.22)
+		(end 60.65 134.22)
 		(width 0.3)
 		(layer "B.Cu")
